Commit message: output

File: assets/panda/panda.urdf (robot description, URDF)
Before this commit: robot panda, 13 links, 12 joints
Joints:
- joint panda_finger_joint1: limit lower=0.0 upper=0.04 effort=20 velocity=0.2 -> (none); origin xyz=0 0 0.0584 rpy=0 0 0 -> xyz=0 0.065 0.0584 rpy=0 0 0; type prismatic -> fixed
- joint panda_finger_joint2: limit lower=0.0 upper=0.04 effort=20 velocity=0.2 -> (none); origin xyz=0 0 0.0584 rpy=0 0 0 -> xyz=0 -0.065 0.0584 rpy=0 0 0; type prismatic -> fixed

File: spherized.urdf (robot description, URDF)
Before this commit: robot panda, 13 links, 12 joints
Links:
- removed link panda_grasptarget
- removed link panda_hand
- removed link panda_leftfinger
- removed link panda_link0
- removed link panda_link1
- removed link panda_link2
- removed link panda_link3
- removed link panda_link4
- removed link panda_link5
- removed link panda_link6
- removed link panda_link7
- removed link panda_link8
- removed link panda_rightfinger
- added link Cube1; collision sphere radius=0.016986; collision sphere radius=0.018471
- added link _builder_root_link
- added link base; collision sphere radius=0.024919; collision sphere radius=0.026381
- added link side_back; collision sphere radius=0.025701; collision sphere radius=0.029479
- added link side_cap; collision sphere radius=0.028583; collision sphere radius=0.029121
- added link side_frontA; collision sphere radius=0.04735; collision sphere radius=0.048381
- added link side_frontB; collision sphere radius=0.04735; collision sphere radius=0.048381
- added link side_left; collision sphere radius=0.022455; collision sphere radius=0.022455
- added link side_right; collision sphere radius=0.025701; collision sphere radius=0.026258
Joints:
- removed joint panda_finger_joint1
- removed joint panda_finger_joint2
- removed joint panda_grasptarget_hand
- removed joint panda_hand_joint
- removed joint panda_joint1
- removed joint panda_joint2
- removed joint panda_joint3
- removed joint panda_joint4
- removed joint panda_joint5
- removed joint panda_joint6
- removed joint panda_joint7
- removed joint panda_joint8
- added joint Cube1_joint: type fixed, parent _builder_root_link, child Cube1
- added joint base_joint: type fixed, parent _builder_root_link, child base
- added joint side_back_joint: type fixed, parent _builder_root_link, child side_back
- added joint side_cap_joint: type fixed, parent _builder_root_link, child side_cap
- added joint side_frontA_joint: type fixed, parent _builder_root_link, child side_frontA
- added joint side_frontB_joint: type fixed, parent _builder_root_link, child side_frontB
- added joint side_left_joint: type fixed, parent _builder_root_link, child side_left
- added joint side_right_joint: type fixed, parent _builder_root_link, child side_right
