Commit message: tuning for fetch

File: assets/fetch/fetch_spherized.urdf (robot description, URDF)
Before this commit: robot fetch, 22 links, 21 joints
Links:
- removed link torso_geo_link_1
- removed link torso_geo_link_2
- link base_link: geometry collision sphere radius=0.119672; collision sphere radius=0.160226
- link elbow_flex_link: geometry collision sphere radius=0.023624; collision sphere radius=0.04463
- link forearm_roll_link: geometry collision sphere radius=0.03138; collision sphere radius=0.034973
- link gripper_link: geometry collision sphere radius=0.003493; collision sphere radius=0.007533
- link head_pan_link: geometry collision sphere radius=0.057197; collision sphere radius=0.062736
- link head_tilt_link: geometry collision sphere radius=0.039413; collision sphere radius=0.041709
- link l_gripper_finger_link: geometry collision sphere radius=0.009531; collision sphere radius=0.009664
- link r_gripper_finger_link: geometry collision sphere radius=0.009203; collision sphere radius=0.009709
- link shoulder_lift_link: geometry collision sphere radius=0.043129; collision sphere radius=0.046071
- link shoulder_pan_link: geometry collision sphere radius=0.041094; collision sphere radius=0.05225
- link torso_fixed_link: geometry collision sphere radius=0.10859; collision sphere radius=0.109413
- link torso_lift_link: geometry collision sphere radius=0.029644; collision sphere radius=0.033433
- link upperarm_roll_link: geometry collision sphere radius=0.038535; collision sphere radius=0.043973
- link wrist_flex_link: geometry collision sphere radius=0.037029; collision sphere radius=0.043566
- link wrist_roll_link: geometry collision sphere radius=0.024466; collision sphere radius=0.025095
Joints:
- removed joint torso_geo_joint_1
- removed joint torso_geo_joint_2
- joint l_gripper_finger_joint: origin xyz=0 -0.015425 0 rpy=0 0 0 -> xyz=0 -0.065425 0 rpy=0 0 0
- joint r_gripper_finger_joint: origin xyz=0 0.015425 0 rpy=0 0 0 -> xyz=0 0.065425 0 rpy=0 0 0

File: assets/fetch/fetch_spherized_1.urdf (robot description, URDF)
Before this commit: robot fetch, 21 links, 20 joints
Links:
- removed link estop_link
- link base_link: geometry collision sphere radius=0.298438; visual mesh filename=package://meshes/base_link.dae
- link elbow_flex_link: geometry collision sphere radius=0.109691; visual mesh filename=package://meshes/elbow_flex_link.dae
- link forearm_roll_link: geometry collision sphere radius=0.112823; visual mesh filename=package://meshes/forearm_roll_link.dae
- link gripper_link: geometry collision sphere radius=0.077127; visual mesh filename=package://meshes/gripper_link.dae
- link head_pan_link: geometry collision sphere radius=0.17117; visual mesh filename=package://meshes/head_pan_link.dae
- link head_tilt_link: geometry collision sphere radius=0.114563; visual mesh filename=package://meshes/head_tilt_link.dae
- link l_gripper_finger_link: geometry collision sphere radius=0.029626; visual mesh filename=package://meshes/l_gripper_finger_link.STL
- link r_gripper_finger_link: geometry collision sphere radius=0.029619; visual mesh filename=package://meshes/r_gripper_finger_link.STL
- link shoulder_lift_link: geometry collision sphere radius=0.11537; visual mesh filename=package://meshes/shoulder_lift_link.dae
- link shoulder_pan_link: geometry collision sphere radius=0.121961; visual mesh filename=package://meshes/shoulder_pan_link.dae
- link torso_fixed_link: geometry collision sphere radius=0.276835; visual mesh filename=package://meshes/torso_fixed_link.dae
- link torso_lift_link: geometry collision sphere radius=0.085846; collision sphere radius=0.103097
- link upperarm_roll_link: geometry collision sphere radius=0.116504; visual mesh filename=package://meshes/upperarm_roll_link.dae
- link wrist_flex_link: geometry collision sphere radius=0.090216; visual mesh filename=package://meshes/wrist_flex_link.dae
- link wrist_roll_link: geometry collision sphere radius=0.051255; visual mesh filename=package://meshes/wrist_roll_link.dae
Joints:
- removed joint estop_joint
- joint forearm_roll_joint: limit effort=29.35 velocity=1.571 -> lower=-3.14159 upper=3.14159 effort=29.35 velocity=1.571; type continuous -> revolute
- joint upperarm_roll_joint: limit effort=76.94 velocity=1.571 -> lower=-3.14159 upper=3.14159 effort=76.94 velocity=1.571; type continuous -> revolute
- joint wrist_roll_joint: limit effort=7.36 velocity=2.268 -> lower=-3.14159 upper=3.14159 effort=7.36 velocity=2.268; type continuous -> revolute
