Commit message: update

File: assets/baxter/baxter.urdf (robot description, URDF)
Before this commit: robot baxter, 61 links, 60 joints
Links:
- removed link l_gripper_l_finger_2
- removed link l_gripper_r_finger_2
- removed link r_gripper_l_finger_2
- removed link r_gripper_r_finger_2
- link head: geometry visual mesh filename=meshes/head/H0.DAE
- link l_gripper_l_finger: geometry collision box size=0.01 0.0135 0.1127; collision box size=0.01 0.05 0.017
- link l_gripper_r_finger: geometry collision box size=0.01 0.0135 0.1127; collision box size=0.01 0.05 0.017
- link r_gripper_l_finger: geometry collision box size=0.01 0.0135 0.1127; collision box size=0.01 0.05 0.017
- link r_gripper_r_finger: geometry collision box size=0.01 0.0135 0.1127; collision box size=0.01 0.05 0.017
- link screen: geometry visual mesh filename=meshes/head/H1.DAE
- link sonar_ring: geometry visual cylinder length=0.01 radius=0.085
- link torso: geometry collision mesh filename=meshes/torso/base_link_collision_1.stl; collision mesh filename=meshes/torso/base_link_collision_2.stl
Joints:
- removed joint l_gripper_l_finger_joint_2
- removed joint l_gripper_r_finger_joint_2
- removed joint r_gripper_l_finger_joint_2
- removed joint r_gripper_r_finger_joint_2
- joint l_gripper_l_finger_joint: origin xyz=0.0 0.019333 0.02 rpy=0 0 0 -> xyz=0.0 0.069333 0.02 rpy=0 0 0
- joint l_gripper_r_finger_joint: origin xyz=0.0 -0.019333 0.02 rpy=0 0 0 -> xyz=0.0 -0.069333 0.02 rpy=0 0 0
- joint r_gripper_l_finger_joint: origin xyz=0.0 0.019333 0.02 rpy=0 0 0 -> xyz=0.0 0.069333 0.02 rpy=0 0 0
- joint r_gripper_r_finger_joint: origin xyz=0.0 -0.019333 0.02 rpy=0 0 0 -> xyz=0.0 -0.069333 0.02 rpy=0 0 0
