Commit message: baxter & fetch

File: spherized.urdf (robot description, URDF)
Before this commit: robot , 9 links, 8 joints
Links:
- removed link Cube1
- removed link _builder_root_link
- removed link base
- removed link side_back
- removed link side_cap
- removed link side_frontA
- removed link side_frontB
- removed link side_left
- removed link side_right
- added link base_link, mass 70.1294; collision sphere radius=0.163736; collision sphere radius=0.172682
- added link elbow_flex_link, mass 2.1299; collision sphere radius=0.045291; collision sphere radius=0.051312
- added link estop_link, mass 0.00196130439134723; collision sphere radius=0.015159; collision sphere radius=0.015908
- added link forearm_roll_link, mass 1.6563; collision sphere radius=0.042387; collision sphere radius=0.042991
- added link gripper_link, mass 1.5175; collision sphere radius=0.049641; collision sphere radius=0.050106
- added link head_camera_depth_frame
- added link head_camera_depth_optical_frame
- added link head_camera_link
- added link head_camera_rgb_frame
- added link head_camera_rgb_optical_frame
- added link head_pan_link, mass 2.2556; collision sphere radius=0.069437; collision sphere radius=0.073477
- added link head_tilt_link, mass 0.9087; collision sphere radius=0.064643; collision sphere radius=0.065906
- added link l_gripper_finger_link, mass 0.0798; collision sphere radius=0.010946; collision sphere radius=0.011177
- added link r_gripper_finger_link, mass 0.0798; collision sphere radius=0.011321; collision sphere radius=0.011455
- added link shoulder_lift_link, mass 2.6615; collision sphere radius=0.05328; collision sphere radius=0.059478
- added link shoulder_pan_link, mass 2.5587; collision sphere radius=0.063705; collision sphere radius=0.064869
- added link torso_fixed_link, mass 13.2775; collision sphere radius=0.036333; collision sphere radius=0.12561
- added link torso_lift_link, mass 10.7796; collision sphere radius=0.09629; collision sphere radius=0.113644
- added link upperarm_roll_link, mass 2.3311; collision sphere radius=0.049454; collision sphere radius=0.052752
- added link wrist_flex_link, mass 1.725; collision sphere radius=0.044337; collision sphere radius=0.053375
- added link wrist_roll_link, mass 0.1354; collision sphere radius=0.023318; collision sphere radius=0.030363
Joints:
- removed joint Cube1_joint
- removed joint base_joint
- removed joint side_back_joint
- removed joint side_cap_joint
- removed joint side_frontA_joint
- removed joint side_frontB_joint
- removed joint side_left_joint
- removed joint side_right_joint
- added joint elbow_flex_joint: type revolute, parent upperarm_roll_link, child elbow_flex_link, origin xyz=0.133 0 0 rpy=0 0 0, axis 0 1 0, limit lower=-2.251 upper=2.251 effort=66.18 velocity=1.521
- added joint estop_joint: type fixed, parent base_link, child estop_link, origin xyz=-0.12465 0.23892 0.31127 rpy=1.5708 0 0, axis 0 0 0
- added joint forearm_roll_joint: type continuous, parent elbow_flex_link, child forearm_roll_link, origin xyz=0.197 0 0 rpy=0 0 0, axis 1 0 0, limit effort=29.35 velocity=1.571
- added joint gripper_axis: type fixed, parent wrist_roll_link, child gripper_link, origin xyz=0.16645 0 0 rpy=0 0 0, axis 0 1 0
- added joint head_camera_depth_joint: type fixed, parent head_camera_link, child head_camera_depth_frame, origin xyz=0 0.045 0 rpy=0 0 0
- added joint head_camera_depth_optical_joint: type fixed, parent head_camera_depth_frame, child head_camera_depth_optical_frame, origin xyz=0 0 0 rpy=-1.57079632679 0 -1.57079632679
- added joint head_camera_joint: type fixed, parent head_tilt_link, child head_camera_link, origin xyz=0.055 0 0.0225 rpy=0 0 0
- added joint head_camera_rgb_joint: type fixed, parent head_camera_link, child head_camera_rgb_frame, origin xyz=0 0.02 0 rpy=0 0 0
- added joint head_camera_rgb_optical_joint: type fixed, parent head_camera_rgb_frame, child head_camera_rgb_optical_frame, origin xyz=0 0 0 rpy=-1.57079632679 0 -1.57079632679
- added joint head_pan_joint: type fixed, parent torso_lift_link, child head_pan_link, origin xyz=0.053125 0 0.603001417713939 rpy=0 0 0, axis 0 0 1
- added joint head_tilt_joint: type fixed, parent head_pan_link, child head_tilt_link, origin xyz=0.14253 0 0.057999 rpy=0 0 0, axis 0 1 0
- added joint l_gripper_finger_joint: type prismatic, parent gripper_link, child l_gripper_finger_link, origin xyz=0 -0.015425 0 rpy=0 0 0, axis 0 -1 0, limit lower=0.0 upper=0.05 effort=60 velocity=0.05
- added joint r_gripper_finger_joint: type prismatic, parent gripper_link, child r_gripper_finger_link, origin xyz=0 0.015425 0 rpy=0 0 0, axis 0 1 0, limit lower=0.0 upper=0.05 effort=60 velocity=0.05
- added joint shoulder_lift_joint: type revolute, parent shoulder_pan_link, child shoulder_lift_link, origin xyz=0.117 0 0.0599999999999999 rpy=0 0 0, axis 0 1 0, limit lower=-1.221 upper=1.518 effort=131.76 velocity=1.454
- added joint shoulder_pan_joint: type revolute, parent torso_lift_link, child shoulder_pan_link, origin xyz=0.119525 0 0.34858 rpy=0 0 0, axis 0 0 1, limit lower=-1.6056 upper=1.6056 effort=33.82 velocity=1.256
- added joint torso_fixed_joint: type fixed, parent base_link, child torso_fixed_link, origin xyz=-0.086875 0 0.377425 rpy=-6.12303176911189E-17 0 0, axis 0 1 0
- added joint torso_lift_joint: type prismatic, parent base_link, child torso_lift_link, origin xyz=-0.086875 0 0.37743 rpy=-6.123E-17 0 0, axis 0 0 1, limit lower=0 upper=0.38615 effort=450.0 velocity=0.1
- added joint upperarm_roll_joint: type continuous, parent shoulder_lift_link, child upperarm_roll_link, origin xyz=0.219 0 0 rpy=0 0 0, axis 1 0 0, limit effort=76.94 velocity=1.571
- added joint wrist_flex_joint: type revolute, parent forearm_roll_link, child wrist_flex_link, origin xyz=0.1245 0 0 rpy=0 0 0, axis 0 1 0, limit lower=-2.16 upper=2.16 effort=25.7 velocity=2.268
- added joint wrist_roll_joint: type continuous, parent wrist_flex_link, child wrist_roll_link, origin xyz=0.1385 0 0 rpy=0 0 0, axis 1 0 0, limit effort=7.36 velocity=2.268

Commit message: Fixes offset by performing transforms in correct order (#3)

File: spherized.urdf (robot description, URDF)
Before this commit: robot fetch, 21 links, 20 joints
Links:
- removed link elbow_flex_link
- removed link estop_link
- removed link forearm_roll_link
- removed link gripper_link
- removed link head_camera_depth_frame
- removed link head_camera_depth_optical_frame
- removed link head_camera_link
- removed link head_camera_rgb_frame
- removed link head_camera_rgb_optical_frame
- removed link head_pan_link
- removed link head_tilt_link
- removed link l_gripper_finger_link
- removed link r_gripper_finger_link
- removed link shoulder_lift_link
- removed link shoulder_pan_link
- removed link torso_fixed_link
- removed link torso_lift_link
- removed link upperarm_roll_link
- removed link wrist_flex_link
- removed link wrist_roll_link
- added link base
- added link base_link_inertia, mass 4.0; collision sphere radius=0.107272; visual mesh filename=package://ur_description/meshes/ur10e/visual/base.dae
- added link flange
- added link forearm_link, mass 3.87; collision sphere radius=0.072633; collision sphere radius=0.077019
- added link shoulder_link, mass 7.778; collision sphere radius=0.122019; visual mesh filename=package://ur_description/meshes/ur10e/visual/shoulder.dae
- added link tool0
- added link upper_arm_link, mass 12.93; collision sphere radius=0.092386; collision sphere radius=0.10311
- added link wrist_1_link, mass 1.96; collision sphere radius=0.079587; visual mesh filename=package://ur_description/meshes/ur10e/visual/wrist1.dae
- added link wrist_2_link, mass 1.96; collision sphere radius=0.081313; visual mesh filename=package://ur_description/meshes/ur10e/visual/wrist2.dae
- added link wrist_3_link, mass 0.202; collision sphere radius=0.052616; visual mesh filename=package://ur_description/meshes/ur10e/visual/wrist3.dae
- link base_link: mass 70.1294 -> None; geometry 
Joints:
- removed joint elbow_flex_joint
- removed joint estop_joint
- removed joint forearm_roll_joint
- removed joint gripper_axis
- removed joint head_camera_depth_joint
- removed joint head_camera_depth_optical_joint
- removed joint head_camera_joint
- removed joint head_camera_rgb_joint
- removed joint head_camera_rgb_optical_joint
- removed joint head_pan_joint
- removed joint head_tilt_joint
- removed joint l_gripper_finger_joint
- removed joint r_gripper_finger_joint
- removed joint torso_fixed_joint
- removed joint torso_lift_joint
- removed joint upperarm_roll_joint
- removed joint wrist_flex_joint
- removed joint wrist_roll_joint
- added joint base_link-base_fixed_joint: type fixed, parent base_link, child base, origin xyz=0 0 0 rpy=0 0 3.141592653589793
- added joint base_link-base_link_inertia: type fixed, parent base_link, child base_link_inertia, origin xyz=0 0 0 rpy=0 0 3.141592653589793
- added joint elbow_joint: type revolute, parent upper_arm_link, child forearm_link, origin xyz=-0.6127 0 0 rpy=0 0 0, axis 0 0 1, limit lower=-3.141592653589793 upper=3.141592653589793 effort=150.0 velocity=3.141592653589793
- added joint flange-tool0: type fixed, parent flange, child tool0, origin xyz=0 0 0 rpy=1.5707963267948966 0 1.5707963267948966
- added joint wrist_1_joint: type revolute, parent forearm_link, child wrist_1_link, origin xyz=-0.57155 0 0.17415 rpy=0 0 0, axis 0 0 1, limit lower=-6.283185307179586 upper=6.283185307179586 effort=56.0 velocity=3.141592653589793
- added joint wrist_2_joint: type revolute, parent wrist_1_link, child wrist_2_link, origin xyz=0 -0.11985 -2.458164590756244e-11 rpy=1.570796327 0 0, axis 0 0 1, limit lower=-6.283185307179586 upper=6.283185307179586 effort=56.0 velocity=3.141592653589793
- added joint wrist_3-flange: type fixed, parent wrist_3_link, child flange, origin xyz=0 0 0 rpy=0 -1.5707963267948966 -1.5707963267948966
- added joint wrist_3_joint: type revolute, parent wrist_2_link, child wrist_3_link, origin xyz=0 0.11655 -2.390480459346185e-11 rpy=1.570796326589793 3.141592653589793 3.141592653589793, axis 0 0 1, limit lower=-6.283185307179586 upper=6.283185307179586 effort=56.0 velocity=3.141592653589793
- joint shoulder_lift_joint: axis 0 1 0 -> 0 0 1; child shoulder_lift_link -> upper_arm_link; limit lower=-1.221 upper=1.518 effort=131.76 velocity=1.454 -> lower=-6.283185307179586 upper=6.283185307179586 effort=330.0 velocity=2.0943951023931953; origin xyz=0.117 0 0.0599999999999999 rpy=0 0 0 -> xyz=0 0 0 rpy=1.570796327 0 0; parent shoulder_pan_link -> shoulder_link
- joint shoulder_pan_joint: child shoulder_pan_link -> shoulder_link; limit lower=-1.6056 upper=1.6056 effort=33.82 velocity=1.256 -> lower=-6.283185307179586 upper=6.283185307179586 effort=330.0 velocity=2.0943951023931953; origin xyz=0.119525 0 0.34858 rpy=0 0 0 -> xyz=0 0 0.1807 rpy=0 0 0; parent torso_lift_link -> base_link_inertia
