Commit message: better spherized xarm6

File: assets/xarm6/xarm6_spherized.urdf (robot description, URDF)
Before this commit: robot xarm6_robot, 20 links, 19 joints
Links:
- link link1: geometry collision sphere radius=0.072604; collision sphere radius=0.08192
- link link2: geometry collision sphere radius=0.055739; collision sphere radius=0.061795
- link link3: geometry collision sphere radius=0.052171; collision sphere radius=0.057715
- link link4: geometry collision sphere radius=0.035913; collision sphere radius=0.040595
- link link5: geometry collision sphere radius=0.057541; collision sphere radius=0.068567
- link link_base: geometry collision sphere radius=0.075535; collision sphere radius=0.089454
