Commit message: working without gripper

File: assets/xarm6/xarm6.urdf (robot description, URDF)
Before this commit: robot xarm6, 20 links, 19 joints
Links:
- removed link left_inner_finger
- removed link left_inner_finger_pad
- removed link left_inner_knuckle
- removed link left_outer_finger
- removed link left_outer_knuckle
- removed link right_inner_finger
- removed link right_inner_finger_pad
- removed link right_inner_knuckle
- removed link right_outer_finger
- removed link right_outer_knuckle
- removed link robotiq_140_base_link
- removed link robotiq_base_link
Joints:
- removed joint finger_joint
- removed joint left_inner_finger_joint
- removed joint left_inner_finger_pad_joint
- removed joint left_inner_knuckle_joint
- removed joint left_outer_finger_joint
- removed joint right_inner_finger_joint
- removed joint right_inner_finger_pad_joint
- removed joint right_inner_knuckle_joint
- removed joint right_outer_finger_joint
- removed joint right_outer_knuckle_joint
- removed joint robotiq_140_base_joint
- removed joint robotiq_base_joint

File: assets/xarm6/xarm6_spherized.urdf (robot description, URDF)
Before this commit: robot xarm6, 20 links, 19 joints
Links:
- removed link left_inner_finger
- removed link left_inner_finger_pad
- removed link left_inner_knuckle
- removed link left_outer_finger
- removed link left_outer_knuckle
- removed link right_inner_finger
- removed link right_inner_finger_pad
- removed link right_inner_knuckle
- removed link right_outer_finger
- removed link right_outer_knuckle
- removed link robotiq_140_base_link
- removed link robotiq_base_link
- link link3: geometry collision sphere radius=0.042045; collision sphere radius=0.046035
- link link5: geometry collision sphere radius=0.056633; collision sphere radius=0.065239
Joints:
- removed joint finger_joint
- removed joint left_inner_finger_joint
- removed joint left_inner_finger_pad_joint
- removed joint left_inner_knuckle_joint
- removed joint left_outer_finger_joint
- removed joint right_inner_finger_joint
- removed joint right_inner_finger_pad_joint
- removed joint right_inner_knuckle_joint
- removed joint right_outer_finger_joint
- removed joint right_outer_knuckle_joint
- removed joint robotiq_140_base_joint
- removed joint robotiq_base_joint
